Commit message: building rl env
temp

lab test done

File: assets/isaac_humanbody_description/urdf/isaac_humanbody.urdf (robot description, URDF)
Before this commit: robot isaac_humanbody, 24 links, 23 joints
Links:
- link l_ankle_dummy1: mass None -> 1e-6
- link l_shoulder_dummy1: mass None -> 1e-6
- link l_shoulder_dummy2: mass None -> 1e-6
- link l_thigh_dummy1: mass None -> 1e-6
- link l_thigh_dummy2: mass None -> 1e-6
- link r_ankle_dummy1: mass None -> 1e-6
- link r_shoulder_dummy1: mass None -> 1e-6
- link r_shoulder_dummy2: mass None -> 1e-6
- link r_thigh_dummy1: mass None -> 1e-6
- link r_thigh_dummy2: mass None -> 1e-6
- link waist_dummy1: mass None -> 1e-6
- link waist_dummy2: mass None -> 1e-6
